File: DS100M08KV2.kicad_sch (KiCad schematic)
At the start: 129 parts, among them J1 wire2board, J10 BNC_panel_mount, J11 wire2board, J2 Conn_01x04_Socket, J3 wire2board, J4 wire2board, J5 USB_C_floating, J8 red_safety_4mm_connector, J9 black_safety_4mm_connector, Q1 BD679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

Commit message: fin
Parts:
- removed C17, C28: 1u, Resistor_SMD:R_0603_1608Metric_Pad0.98x0.95mm_HandSolder, symbol Device:C
- removed C40: 47u, Capacitor_THT:CP_Radial_D5.0mm_P2.00mm, symbol Device:C_Polarized_US
- removed L2: 4.7u, Inductor_THT:L_Radial_D7.5mm_P3.50mm_Fastron_07P, symbol Device:L
- removed L3: 4.7u, Inductor_SMD:L_Bourns_SRN6045TA, symbol Device:L
- removed PS1: IA0509S, Converter_DCDC:Converter_DCDC_XP_POWER-IAxxxxS_THT, symbol Converter_DCDC:IA0509S
- removed Q1: BD679, Package_TO_SOT_THT:TO-126-3_Vertical, symbol DS100M06V_linear:BD679
- removed Q4: BD680, Package_TO_SOT_THT:TO-126-3_Vertical, symbol DS100M06V_linear:BD680
- removed U7: TLV61070ADBVR, Package_TO_SOT_SMD:SOT-23-6, symbol DS100M08KV:TLV61070ADBVR
- added D8: 1N4148W, Diode_SMD:D_SOD-123, symbol Diode:1N4148W
- added Q1, Q9: MMBT3906, Package_TO_SOT_SMD:SOT-23, symbol Transistor_BJT:MMBT3906
- added Q10, Q8: AO3401A, Package_TO_SOT_SMD:SOT-23, symbol Transistor_FET:AO3401A
- added Q13, Q14: AO3400A, Package_TO_SOT_SMD:SOT-23, symbol Transistor_FET:AO3400A
- added Q2, Q6: MMBT5551L, Package_TO_SOT_SMD:SOT-23, symbol Transistor_BJT:MMBT5551L
- C41, C42, C43: footprint Resistor_SMD:R_1206_3216Metric_Pad1.30x1.75mm_HandSolder -> Resistor_SMD:R_0603_1608Metric_Pad0.98x0.95mm_HandSolder
- R27: value 10k -> 22k; LCSC (none) -> C31850
- R28: value 91k -> 81k
- R32: value 2k2 -> 22k; LCSC (none) -> C31850
- R34: value 2k2 -> 81k
Connections:
- net +5V: no longer C31.1, C44.1
- net -5V: no longer C30.1, C36.2
- net -BAT: now also C43.1, D8.1 (K), Q10.2 (S), Q13.2 (S)
- net 0: now also R27.2, R32.2, Q6.2 (E), Q9.2 (E); no longer R32.1, R34.1
- net Earth: no longer C41.1, C42.1, C43.1, R27.1
- net +VIN: now reaches C3.1, R31.2
- net +VIN: now also SW2.2 (B), Q2.3 (C), Q8.2 (S)
- net -VIN: now reaches C43.2
- net -VIN: now also C29.1, R33.2, Q1.3 (C), Q14.2 (S); no longer SW2.2 (B)
- net at C20.2, R33.1: now also R34.1, Q1.1 (B), Q9.3 (C); no longer R34.2
- net at C16.1, R31.1: now also R28.1, Q2.1 (B), Q6.3 (C); no longer R32.2
- removed net +5V_BOOST: C41.2, C42.2, R28.2
- new net: Q9.1 (B), R32.1, R34.2
- new net: Q6.1 (B), R27.1, R28.2
- new net: C42.1, D8.2 (A), Q10.1 (G), Q14.1 (G)
- new net: C41.1, Q13.3 (D), Q8.3 (D)
- new net: C41.2, Q10.3 (D), Q14.3 (D)
- new net +2.5V: C31.1, C44.1, Q2.2 (E)
- new net -2.5V: C30.1, C36.2, Q1.2 (E)
- new net GATE: C42.2, Q13.1 (G), Q8.1 (G)
Other:
- moved on the sheet: C16, C20, C29, C3, C30, C31, C36, C44, R31, R33

Commit message: new osc.
Parts:
- removed C1, C27: 1u, Resistor_SMD:R_0603_1608Metric_Pad0.98x0.95mm_HandSolder, symbol Device:C
- removed C33: 100n, Resistor_SMD:R_0603_1608Metric_Pad0.98x0.95mm_HandSolder, symbol Device:C
- removed C34: 1n, Resistor_SMD:R_0603_1608Metric_Pad0.98x0.95mm_HandSolder, symbol Device:C
- added C17: 1n, Capacitor_SMD:C_0603_1608Metric_Pad1.08x0.95mm_HandSolder, symbol Device:C
- added C28, C47: 100n, Capacitor_SMD:C_0603_1608Metric_Pad1.08x0.95mm_HandSolder, symbol Device:C
- added C40, C46: 1u, Capacitor_SMD:C_0603_1608Metric_Pad1.08x0.95mm_HandSolder, symbol Device:C
- added D10, D9: 1N4148WS, Diode_SMD:D_SOD-323, symbol Diode:1N4148WS
- added R19: 39k, Resistor_SMD:R_0603_1608Metric_Pad0.98x0.95mm_HandSolder, symbol Device:R
- added R21, R39: 470k, Resistor_SMD:R_0603_1608Metric_Pad0.98x0.95mm_HandSolder, symbol Device:R
- added R37, R38: 100k, Resistor_SMD:R_0603_1608Metric_Pad0.98x0.95mm_HandSolder, symbol Device:R
- added U3: 74HC14D653, Package_SO:SOIC-14_3.9x8.7mm_P1.27mm, symbol 74xx:74HC14
- C18: value 100n -> 10u; footprint Resistor_SMD:R_0603_1608Metric_Pad0.98x0.95mm_HandSolder -> Capacitor_SMD:C_0603_1608Metric_Pad1.08x0.95mm_HandSolder; LCSC (none) -> C96446
- C19: value 1u -> 10u; footprint Resistor_SMD:R_0603_1608Metric_Pad0.98x0.95mm_HandSolder -> Capacitor_SMD:C_0603_1608Metric_Pad1.08x0.95mm_HandSolder; LCSC (none) -> C96446
- C35: value 1n -> 100n; footprint Resistor_SMD:R_0603_1608Metric_Pad0.98x0.95mm_HandSolder -> Capacitor_SMD:C_0603_1608Metric_Pad1.08x0.95mm_HandSolder; LCSC (none) -> C14663
- C45: footprint Resistor_SMD:R_0603_1608Metric_Pad0.98x0.95mm_HandSolder -> Capacitor_SMD:C_0603_1608Metric_Pad1.08x0.95mm_HandSolder; LCSC (none) -> C14663
Connections:
- net +VBUS: now also C28.2, C40.2; no longer C45.1
- net +VIN: now also C45.2, C46.2, U3.14 (VCC)
- net -BAT: now also C45.1, C46.1, U3.7 (GND)
- net 0: now also C18.2, C19.2, C17.1, C47.1; no longer C18.1, C19.1
- net Earth: now also C28.1, C40.1; no longer C45.2
- net GATE: now also U3.10, U3.12, U3.4, U3.6, U3.8
- net at C35.2, FB1.1, U1.4 (V-): now also C18.1; no longer C18.2
- net at FB2.1, U1.8 (V+): now also C19.1, C47.2; no longer C19.2
- new net: D10.2 (A), R38.2, R39.2
- new net: D9.1 (K), R21.2, R37.2
- new net: C17.2, R19.2, R21.1, R37.1, R38.1, R39.1, U3.1
- new net CLK: D10.1 (K), D9.2 (A), R19.1, U3.11, U3.13, U3.2, U3.3, U3.5, U3.9
Other:
- moved on the sheet: FB2

Commit message: New sims, added switcher to PCB.
Parts:
- removed BT1: Battery_Cell, DS100M08KV:battery_holder, symbol Device:Battery_Cell
- removed C16, C20, C36, C44: 47u, Capacitor_THT:CP_Radial_D5.0mm_P2.00mm, symbol Device:C_Polarized_US
- removed C17: 1n, Capacitor_SMD:C_0603_1608Metric_Pad1.08x0.95mm_HandSolder, symbol Device:C
- removed C2: 100n, Resistor_SMD:R_0603_1608Metric_Pad0.98x0.95mm_HandSolder, symbol Device:C
- removed C28, C45: 100n, Capacitor_SMD:C_0603_1608Metric_Pad1.08x0.95mm_HandSolder, symbol Device:C
- removed C29, C3, C30, C31: 1u, Resistor_SMD:R_0603_1608Metric_Pad0.98x0.95mm_HandSolder, symbol Device:C
- removed C40, C46: 1u, Capacitor_SMD:C_0603_1608Metric_Pad1.08x0.95mm_HandSolder, symbol Device:C
- removed C41, C42, C43: 10u, Resistor_SMD:R_0603_1608Metric_Pad0.98x0.95mm_HandSolder, symbol Device:C
- removed D10, D9: 1N4148WS, Diode_SMD:D_SOD-323, symbol Diode:1N4148WS
- removed D6: LED, LED_THT:LED_D3.0mm_FlatTop, symbol Device:LED
- removed D8: 1N4148W, Diode_SMD:D_SOD-123, symbol Diode:1N4148W
- removed J2: Conn_01x04_Socket, Connector_JST:JST_PH_B4B-PH-K_1x04_P2.00mm_Vertical, symbol Connector:Conn_01x04_Socket
- removed J5: USB_C_floating, DS100M08KV:USB_C_floating, symbol DS100M08KV:USB_C_floating
- removed Q1, Q9: MMBT3906, Package_TO_SOT_SMD:SOT-23, symbol Transistor_BJT:MMBT3906
- removed Q10, Q8: AO3401A, Package_TO_SOT_SMD:SOT-23, symbol Transistor_FET:AO3401A
- removed Q13, Q14: AO3400A, Package_TO_SOT_SMD:SOT-23, symbol Transistor_FET:AO3400A
- removed Q2, Q6: MMBT5551L, Package_TO_SOT_SMD:SOT-23, symbol Transistor_BJT:MMBT5551L
- removed Q3, Q5: CMSN3416K-HF, Package_TO_SOT_SMD:SOT-23, symbol Transistor_FET:BSS123
- removed R19: 39k, Resistor_SMD:R_0603_1608Metric_Pad0.98x0.95mm_HandSolder, symbol Device:R
- removed R21, R39: 470k, Resistor_SMD:R_0603_1608Metric_Pad0.98x0.95mm_HandSolder, symbol Device:R
- removed R25, R36: 10k, Resistor_SMD:R_0603_1608Metric_Pad0.98x0.95mm_HandSolder, symbol Device:R
- removed R26, R30: 330, Resistor_SMD:R_0603_1608Metric_Pad0.98x0.95mm_HandSolder, symbol Device:R
- removed R27, R32: 22k, Resistor_SMD:R_0603_1608Metric_Pad0.98x0.95mm_HandSolder, symbol Device:R
- removed R28, R34: 81k, Resistor_SMD:R_0603_1608Metric_Pad0.98x0.95mm_HandSolder, symbol Device:R
- removed R29: 2.7k, Resistor_SMD:R_0603_1608Metric_Pad0.98x0.95mm_HandSolder, symbol Device:R
- removed R31, R33: 1k, Resistor_SMD:R_0603_1608Metric_Pad0.98x0.95mm_HandSolder, symbol Device:R
- removed R37, R38: 100k, Resistor_SMD:R_0603_1608Metric_Pad0.98x0.95mm_HandSolder, symbol Device:R
- removed SW2: SW_DPDT_x2, DS100M08KV:DPDT_bigger, symbol Switch:SW_DPDT_x2
- removed U2: AP9101CK6, Package_TO_SOT_SMD:SOT-23-6, symbol Battery_Management:AP9101CK6
- removed U3: 74HC14D653, Package_SO:SOIC-14_3.9x8.7mm_P1.27mm, symbol 74xx:74HC14
- removed U6: BQ21040DBV, Package_TO_SOT_SMD:SOT-23-6, symbol Battery_Management:BQ21040DBV
- D2, D7: LCSC (none) -> C2500; now not fitted
Connections:
- no-connect marks 2 -> 0
Other:
- added sheet Power supply (power_supply.kicad_sch)

Commit message: Sims, schem.
Parts:
- removed FB3, FB4: FerriteBead, Inductor_SMD:L_0603_1608Metric_Pad1.05x0.95mm_HandSolder, symbol Device:FerriteBead
- removed RV4: 100k, Potentiometer_THT:Potentiometer_Bourns_3296W_Vertical, symbol Device:R_Potentiometer
- removed U4: AD8009, Package_SO:SOIC-8_3.9x4.9mm_P1.27mm, symbol DS100M08KV:AD8009
- added C56: 100p, Resistor_SMD:R_0603_1608Metric_Pad0.98x0.95mm_HandSolder, symbol Device:C
- added C57, C58: 10p, Resistor_SMD:R_0603_1608Metric_Pad0.98x0.95mm_HandSolder, symbol Device:C
- added R31, R54: 100, Resistor_SMD:R_0603_1608Metric_Pad0.98x0.95mm_HandSolder, symbol Device:R
- added R53: 200, Resistor_SMD:R_0603_1608Metric_Pad0.98x0.95mm_HandSolder, symbol Device:R
- C21, C22, C4: value 100n -> 330p; LCSC (none) -> C1664
- C23, C24, C25, C37: value 1n -> 100p; LCSC (none) -> C14858
- C26: value 1u -> 100p; LCSC (none) -> C14858
- C32, C7, C8: footprint Resistor_SMD:R_0603_1608Metric_Pad0.98x0.95mm_HandSolder -> Capacitor_SMD:C_0603_1608Metric_Pad1.08x0.95mm_HandSolder; LCSC (none) -> C14663
- C38: value 100n -> 100p; LCSC (none) -> C14858
- C5: value 470p -> 330p; LCSC (none) -> C1664
- C6: value 470p -> 100p; LCSC (none) -> C14858
- R12, R5: value 5k -> 10k
- R13: value 50 -> 82k
- R14, R15: LCSC (none) -> C25803
- R16: value 10 -> 10k
- R17, R35, R51, R52: LCSC (none) -> C22775
- R18: value 1k -> 82k
- R20: value 100 -> 200
- R23, R7: LCSC (none) -> C7250
- R24: value 51k -> 200
- R6: value 500 -> 10k
- U1: LCSC (none) -> RS8752XK
Connections:
- net 0: now also C21.2, C22.2, C4.2, C5.2, R24.2; no longer C21.1, C22.1, C25.1, C4.1, C5.1, R22.2
- net at SW1.3 (C): now also R54.2; no longer R20.1
- net at R17.2, R35.1: now also R20.2, U1.1; no longer R18.2
- net at C26.2, C37.2: now also C38.2, C4.1, C5.1, C8.1, R12.2, R16.2, R51.2, C56.2, C58.2; no longer C21.2
- net at D2.3 (K), U1.5 (+): now also SW1.5 (B); no longer R52.1
- net at SW1.1 (A): now also R31.1; no longer R16.1
- net at R13.2: now also R6.1; no longer SW1.6 (C)
- net at R24.1: now also U1.6 (-), R53.2; no longer C4.2
- net at D4.1 (K), D5.1 (K), R14.1: now also C8.2; no longer C8.1
- net at R6.2: now also C11.1, C25.2, R3.2, R7.1, TP1.1, C57.2, R31.2; no longer SW1.4 (A)
- net at D7.3 (K), U1.3 (+): now also SW1.2 (B); no longer R51.1
- new net: R51.1, SW1.4 (A)
- new net: C15.1, C56.1, C58.1, R11.2, R18.1, R23.1, R52.1, TP2.1
- new net: C21.1, C22.1, C23.2, C24.2, C25.1, C57.1, C6.2, C7.2, R13.1, R5.2, R54.1
- new net: R22.1, R53.1, U1.7
- new net: R20.1, R22.2, U1.2 (-)
- new net: R52.2, SW1.6 (C)
- new net: R16.1, R18.2
Other:
- note added: "https://www.digikey.com/en/products/detail/texas-instruments/TLV3542IDR/6553879"
- note removed: "for best BW, 200 Ohm highest for 100 MHz , 1 kOhm"
- moved on the sheet: C12, C13, C14, C15, C18, C19, C35, C47, C6, D1, D2, D3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

Commit message: Placement done.
Parts:
- removed H2: MountingHole, DS100M08KV:M3_with_screw, symbol Mechanical:MountingHole
- removed TP3, TP4: TestPoint, TestPoint:TestPoint_Pad_D2.0mm, symbol Connector:TestPoint
- added C66, C67: 100n, Capacitor_SMD:C_0603_1608Metric_Pad1.08x0.95mm_HandSolder, symbol Device:C
Connections:
- net -5V is gone; now on net -2V5: D2.1 (K), D7.1 (K), FB1.2, RV1.1
- net +2V5: now also D2.2 (A), D7.2 (A), FB2.2, RV1.3, RV5.3
- net 0: now also C66.1, C67.1
- net at R51.1: now also SW1.6 (C); no longer SW1.4 (A)
- net at R24.1, R53.2: now also U1.2 (-); no longer U1.6 (-)
- net at D2.3 (K), SW1.5 (B): now also U1.3 (+); no longer U1.5 (+)
- net at R22.1, R53.1: now also U1.1; no longer U1.7
- net at R15.2, RV5.2: now also C66.2
- net at SW1.1 (A): now also R54.2; no longer R31.1
- net at D7.3 (K), SW1.2 (B): now also U1.5 (+); no longer U1.3 (+)
- net at SW1.3 (C): now also R31.1; no longer R54.2
- net at R20.1, R22.2: now also U1.6 (-); no longer U1.2 (-)
- net at R14.2, RV6.2: now also C67.2
- net at R17.2, R20.2, R35.1: now also U1.7; no longer U1.1
- net at R52.2: now also SW1.4 (A); no longer SW1.6 (C)
- removed net +5V: D2.2 (A), D7.2 (A), FB2.2, RV1.3, RV5.3, RV6.3
Other:
- moved on the sheet: C7, C8, D1, D3, D4, D5, R14, R15, RV5, RV6, SW1A, SW1B
