File: DS100M08KV2.kicad_pcb (KiCad board)
At the start: 4 copper layers, 100 x 52 mm, 180 parts, among them J1 wire2board, J10 BNC_panel_mount, J11 wire2board, J2 Conn_01x04_Socket, J3 wire2board, J4 wire2board, J5 USB_C_floating, J8 red_safety_4mm_connector, J9 black_safety_4mm_connector, Q1 MMBT5401, Q10 AO3401A, Q13 AO3400A, Q14 AO3400A, Q2 MMBT5551L, Q3 CMSN3416K-HF, Q4 MMBT5401, Q5 CMSN3416K-HF, Q6 MMBT5551L, Q8 AO3401A, SW1 SW_DPDT_x2, SW2 SW_DPDT_x2, U1 RS8752XK, U2 AP9101CK6, U3 74HC14D653, U4 TL431DBZ, U6 BQ21040DBV

Commit message: Amp.
Parts:
- moved C35 3.50 mm to (141.5, 118.5), turned to 0 degrees
- moved C18 0.94 mm to (144.1, 120.5), turned to -90 degrees
Routing:
- net +BATT: track 2.60 -> 74.3 mm, vias 0 -> 1
- net +2V5: track 14.9 -> 82.8 mm, vias 0 -> 4
- net -2V5: track 9.57 -> 70.1 mm, vias 0 -> 4
- net 0: track 44.1 -> 73.9 mm, vias 23 -> 27
- net Net-(C66-Pad2): track 0.00 -> 17.9 mm, vias 0 -> 2
- net Net-(U1B--): track 0.00 -> 8.20 mm
- net Net-(SW1A-A): track 0.00 -> 7.85 mm
- net Net-(U1C-V-): track 0.00 -> 6.39 mm
- net Net-(R17-Pad2): track 0.00 -> 5.23 mm
- net Net-(U1C-V+): track 0.00 -> 4.76 mm
- net Net-(J1-Pin_1): track 0.00 -> 3.91 mm
- net Net-(R22-Pad1): track 0.00 -> 3.80 mm
- net Net-(U1A--): track 0.00 -> 3.62 mm
