File: DS100M08KV2.kicad_pcb (KiCad board)
At the start: 4 copper layers, 100 x 52 mm, 180 parts, among them J1 wire2board, J10 BNC_panel_mount, J11 wire2board, J2 Conn_01x04_Socket, J3 wire2board, J4 wire2board, J5 USB_C_floating, J8 red_safety_4mm_connector, J9 black_safety_4mm_connector, Q1 MMBT5401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

Commit message: Almost done.
Parts:
- moved C28 14.0 mm to (131.7, 145.4), turned to 0 degrees
- moved C32 8.49 mm to (131.2, 116.0), turned to 180 degrees
- moved TP1 4.55 mm to (125.9, 113.6)
- moved R7 4.14 mm to (127.7, 116.7), turned to 0 degrees
- turned C40 to 90 degrees
Connections:
- C1 pad 1: -BATT -> Earth
- C17 pad 1: -BATT -> Earth
- C2 pad 2: Earth -> -BATT
- C31 pad 1: -BATT -> Earth
- C33 pad 1: -BATT -> Earth
- C34 pad 1: -BATT -> Earth
- C45 pad 1: -BATT -> Earth
- C46 pad 1: -BATT -> Earth
- C51 pad 1: -BATT -> Earth
- C52 pad 1: -BATT -> Earth
- C53 pad 1: -BATT -> Earth
- C54 pad 1: -BATT -> Earth
- C59 pad 1: -BATT -> Earth
- C63 pad 1: -BATT -> Earth
- C64 pad 1: -BATT -> Earth
- D8 pad 1: -BATT -> Earth
- Q10 pad 2: -BATT -> Earth
- Q13 pad 2: -BATT -> Earth
- Q3 pad 2: Earth -> -BATT
- Q5 pad 2: -BATT -> Earth
- R29 pad 1: -BATT -> Earth
- R30 pad 1: +BAT -> +BATT
- U2 pad 6: Earth -> -BATT
- U3 pad 7: -BATT -> Earth
- U6 pad 2: +BAT -> -BATT
Routing:
- net -BATT: track 37.3 -> 99.8 mm, vias 11 -> 4
- net Earth: track 13.2 -> 41.4 mm, vias 5 -> 14
- net +BAT: track 19.1 -> 0.00 mm, vias 2 -> 0
- net +BATT: track 74.3 -> 88.7 mm, vias 1 -> 2
- net +VBUS: track 6.36 -> 17.3 mm
- net Net-(Q1-B): track 21.3 -> 25.8 mm
- net Net-(U2-VM): track 0.00 -> 3.99 mm
- net Net-(Q3-D): track 0.00 -> 3.90 mm
- net Net-(U2-VDD): track 0.00 -> 3.66 mm
- net Net-(C32-Pad2): track 9.46 -> 13.0 mm
- net Net-(Q3-G): track 0.00 -> 3.31 mm
- net Net-(Q5-G): track 0.00 -> 2.48 mm
- net 0: track 73.9 -> 71.4 mm
- net Net-(C11-Pad1): track 16.4 -> 16.7 mm, vias 1 -> 0
- added copper zone on B.Cu, net Earth
- added copper zone on F.Cu, net Earth
- removed copper zone on B.Cu, net -BATT
- removed copper zone on F.Cu, net -BATT

Commit message: Skoro gotovo Skoro gotovo
Routing:
- net -BATT: track 99.8 -> 97.2 mm
- net -2V5: track 70.1 -> 68.0 mm
- net +VIN: track 87.6 -> 86.3 mm
- net +2V5: track 82.8 -> 81.8 mm
- net 0: track 71.4 -> 70.5 mm
- net +BATT: track 88.7 -> 87.9 mm
- net Net-(SW1B-B): track 18.1 -> 17.4 mm
- net Net-(Q1-B): track 25.8 -> 26.4 mm
- net Net-(SW1A-C): track 22.3 -> 21.7 mm
- net /Power supply/MID_REC: track 16.7 -> 16.2 mm
- net Net-(D12-A): track 24.8 -> 25.3 mm
- net -VIN: track 72.9 -> 72.4 mm
Other:
- board text added: "+"
- board text added: "-"
- board text added: "CAP COMP"
- board text added: "DC OFFSET"
- board text added: "G"

Commit message: Bom
Parts:
- C2: footprint Resistor_SMD:R_0603_1608Metric_Pad0.98x0.95mm_HandSolder -> Capacitor_SMD:C_0603_1608Metric_Pad1.08x0.95mm_HandSolder
- D13, D8: value 1N4148W -> 1N4148WS; footprint Diode_SMD:D_SOD-123 -> Diode_SMD:D_SOD-323
- Q3, Q5: value CMSN3416K-HF -> AO3400A
- R26: value 330 -> 1k
- moved D8 0.10 mm to (180.9, 147.6)
- turned C2 to 90 degrees
- turned R25 to 90 degrees
- turned R36 to 0 degrees
Connections:
- C2 pad 1: Net-(U2-VDD) -> -BATT
- C2 pad 2: -BATT -> Net-(U2-VDD)
- R25 pad 1: Earth -> Net-(U6-TS)
- R25 pad 2: Net-(U6-TS) -> Earth
- R36 pad 1: Earth -> Net-(U6-ISET)
- R36 pad 2: Net-(U6-ISET) -> Earth
Routing:
- net Net-(D8-A): track 4.29 -> 4.99 mm
- net -BATT: track 97.2 -> 97.9 mm
- net Net-(D13-A): track 9.61 -> 10.2 mm
Other:
- copper layers 4 -> 2
