File: power_supply.kicad_sch (KiCad schematic)
At the start: 78 parts, among them J2 Conn_01x04_Socket, J5 USB_C_floating, Q1 MMBT5401, Q10 AO3401A, Q13 AO3400A, Q14 AO3400A, Q2 MMBT5551L, Q3 CMSN3416K-HF, Q4 MMBT5401, Q5 CMSN3416K-HF, Q6 MMBT5551L, Q8 AO3401A, SW2 SW_DPDT_x2, U2 AP9101CK6, U3 74HC14D653, U6 BQ21040DBV

Commit message: Layout
Parts:
- added C31, C59, C60: 100n, Capacitor_SMD:C_0603_1608Metric_Pad1.08x0.95mm_HandSolder, symbol Device:C
- added C61, C62, C63, C64: 47u, Capacitor_THT:CP_Radial_D5.0mm_P2.00mm, symbol Device:C_Polarized_US
- added C65: 10u, Resistor_SMD:R_0805_2012Metric_Pad1.20x1.40mm_HandSolder, symbol Device:C
Connections:
- net +VIN: now also C31.2
- net -BATT: now also C31.1, C59.1, C63.1, C64.1
- net -VIN: now also C59.2, C63.2, C64.2
- net CLK: now also R38.2, R39.2, U3.8; no longer D10.1 (K), U3.2
- net PMOS_GATE: now also U3.2; no longer U3.8
- net MID_DRV: now reaches C41.1, C43.1, C48.1, C49.1, C50.1, Q13.3 (D), Q8.3 (D)
- net MID_DRV: now also C60.2, C61.1, C62.1, C65.1
- net MID_REC: now reaches C41.2, C43.2, C48.2, C49.2, C50.2, Q10.3 (D), Q14.3 (D)
- net MID_REC: now also C60.1, C61.2, C62.2, C65.2
- net at C34.2, D12.2 (A), R42.1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: now also U3.1; no longer U3.9
- net at C17.2, R19.2, R21.1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: now also D10.2 (A), U3.9; no longer R38.1, R39.1, U3.1
- new net: D10.1 (K), R38.1, R39.1
Other:
- moved on the sheet: D10, R38, R39

Commit message: Placement done.
Parts:
- added R55: 1k, Resistor_SMD:R_0603_1608Metric_Pad0.98x0.95mm_HandSolder, symbol Device:R
- added R56: 10k, Resistor_SMD:R_0603_1608Metric_Pad0.98x0.95mm_HandSolder, symbol Device:R
- added TP3, TP4, TP6, TP7, TP8, TP9: TestPoint, TestPoint:TestPoint_Pad_D2.0mm, symbol Connector:TestPoint
- added U4: TL431DBZ, Package_TO_SOT_SMD:SOT-23, symbol Reference_Voltage:TL431DBZ
Connections:
- net +2.5V: now also R55.2
- net +VIN: now also TP7.1
- net -VIN: now also TP9.1
- net 0: now also R56.2, TP6.1, TP8.1, U4.3 (A)
- net at C16.1, Q2.1 (B), Q6.3 (C)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: now also U4.1 (K)
- new net: R55.1, R56.1, U4.2 (REF)
- new net +2V5: TP3.1
- new net -2V5: TP4.1
Other:
- moved on the sheet: C29, C44

Commit message: Switcher done.
Connections:
- net -BAT is gone; now on net -BATT: Q5.2 (S), R29.1
Changed lines of the file:
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@@
 		)
 	)
-	(global_label "-BAT"
-		(shape input)
-		(at 245.11 264.16 0)
-		(fields_autoplaced yes)
-		(effects
-			(font
-				(size 1.27 1.27)
-			)
-			(justify left)
-		)
-		(property "Intersheetrefs" "${INTERSHEET_REFS}"
-			(at 252.9938 264.16 0)
-			(effects
-				(font
-					(size 1.27 1.27)
-				)
-				(justify left)
-				(hide yes)
-			)
-		)
-	)
 	(global_label "+BAT"
 		(shape output)
@@
 					(unit 1)
 				)
+			)
+		)
+	)
+	(symbol
+		(lib_id "power:-BATT")
+		(at 245.11 264.16 270)
+		(unit 1)
+		(exclude_from_sim no)
+		(in_bom yes)
+		(on_board yes)
+		(dnp no)
+		(fields_autoplaced yes)
+		(property "Reference" "#PWR051"
+			(at 241.3 264.16 0)
+			(effects
+				(font
+					(size 1.27 1.27)
+				)
+				(hide yes)
+			)
+		)
+		(property "Value" "-BATT"
+			(at 248.92 264.1599 90)
+			(effects
+				(font
+					(size 1.27 1.27)
+				)
+				(justify left)
+			)
+		)
+		(property "Footprint" ""
+			(at 245.11 264.16 0)
+			(effects
+				(font
+					(size 1.27 1.27)
+				)
+				(hide yes)
+			)
+		)
+		(property "Datasheet" ""
+			(at 245.11 264.16 0)
+			(effects
+				(font
+					(size 1.27 1.27)
+				)
+				(hide yes)
+			)
+		)
+		(property "Description" "Power symbol creates a global label with name \"-BATT\""
+			(at 245.11 264.16 0)
+			(effects
+				(font
+					(size 1.27 1.27)
+				)
+				(hide yes)
+			)
+		)
+		(pin "1"
+		)
+		(instances
+			(project "DS100M08KV2"
+				(path "/e034a6c3-9973-4355-8043-c1e988e27610/78b47647-b6ba-4d31-8265-f09819a98295"
+					(reference "#PWR051")
+					(unit 1)
+				)

Commit message: Lin Reg.
Connections:
- net +BATT: now also SW2.4 (A)
- net +VIN: now also SW2.5 (B)
Changed lines of the file:
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@@
 	(wire
 		(pts
+			(xy 356.87 63.5) (xy 361.95 63.5)
+		)
+		(stroke
+			(width 0)
+			(type default)
+		)
+	)
+	(wire
+		(pts
 			(xy 251.46 48.26) (xy 256.54 48.26)
 		)
@@
 	(wire
 		(pts
+			(xy 372.11 66.04) (xy 375.92 66.04)
+		)
+		(stroke
+			(width 0)
+			(type default)
+		)
+	)
+	(wire
+		(pts
 			(xy 113.03 231.14) (xy 113.03 233.68)
 		)
@@
 		(lib_id "Switch:SW_DPDT_x2")
 		(at 367.03 66.04 0)
+		(mirror y)
 		(unit 2)
 		(exclude_from_sim no)
@@
 	)
 	(symbol
+		(lib_id "power:+BATT")
+		(at 356.87 63.5 90)
+		(unit 1)
+		(exclude_from_sim no)
+		(in_bom yes)
+		(on_board yes)
+		(dnp no)
+		(property "Reference" "#PWR053"
+			(at 360.68 63.5 0)
+			(effects
+				(font
+					(size 1.27 1.27)
+				)
+				(hide yes)
+			)
+		)
+		(property "Value" "+BATT"
+			(at 350.012 63.5 90)
+			(effects
+				(font
+					(size 1.27 1.27)
+				)
+			)
+		)
+		(property "Footprint" ""
+			(at 356.87 63.5 0)
+			(effects
+				(font
+					(size 1.27 1.27)
+				)
+				(hide yes)
+			)
+		)
+		(property "Datasheet" ""
+			(at 356.87 63.5 0)
+			(effects
+				(font
+					(size 1.27 1.27)
+				)
+				(hide yes)
+			)
+		)
+		(property "Description" "Power symbol creates a global label with name \"+BATT\""
+			(at 356.87 63.5 0)
+			(effects
+				(font
+					(size 1.27 1.27)
+				)
+				(hide yes)
+			)
+		)
+		(pin "1"
+		)
+		(instances
+			(project "DS100M08KV2"
+				(path "/e034a6c3-9973-4355-8043-c1e988e27610/78b47647-b6ba-4d31-8265-f09819a98295"
+					(reference "#PWR053")
+					(unit 1)
+				)
+			)
+		)
+	)
+	(symbol
 		(lib_id "Device:R")
 		(at 238.76 154.94 180)
@@
 					(unit 1)
 				)
+			)
+		)
+	)
+	(symbol
+		(lib_id "power:+BATT")
+		(at 375.92 66.04 270)
+		(unit 1)
+		(exclude_from_sim no)
+		(in_bom yes)
+		(on_board yes)
+		(dnp no)
+		(fields_autoplaced yes)
+		(property "Reference" "#PWR052"
+			(at 372.11 66.04 0)
+			(effects
+				(font
+					(size 1.27 1.27)
+				)
+				(hide yes)
+			)
+		)
+		(property "Value" "+VIN"
+			(at 379.73 66.0399 90)
+			(effects
+				(font
+					(size 1.27 1.27)
+				)
+				(justify left)
+			)
+		)
+		(property "Footprint" ""
+			(at 375.92 66.04 0)
+			(effects
+				(font
+					(size 1.27 1.27)
+				)
+				(hide yes)
+			)
+		)
+		(property "Datasheet" ""
+			(at 375.92 66.04 0)
+			(effects
+				(font
+					(size 1.27 1.27)
+				)
+				(hide yes)
+			)
+		)
+		(property "Description" "Power symbol creates a global label with name \"+BATT\""
+			(at 375.92 66.04 0)
+			(effects
+				(font
+					(size 1.27 1.27)
+				)
+				(hide yes)
+			)
+		)
+		(pin "1"
+		)
+		(instances
+			(project "DS100M08KV2"
+				(path "/e034a6c3-9973-4355-8043-c1e988e27610/78b47647-b6ba-4d31-8265-f09819a98295"
+					(reference "#PWR052")
+					(unit 1)
+				)

Commit message: Almost done.
Connections:
- net +BATT: now also R30.1
- net -BATT: now also C2.2, Q3.2 (S), U2.6 (VSS), U6.2 (OUT); no longer C1.1, C17.1, C31.1, C33.1, C34.1, C45.1, C46.1, C51.1, C52.1, C53.1, C54.1, C59.1, C63.1, C64.1, D8.1 (K), Q10.2 (S), Q13.2 (S), Q5.2 (S), R29.1, U3.7 (GND)
- net Earth: now also C1.1, C17.1, C31.1, C33.1, C34.1, C45.1, C46.1, C51.1, C52.1, C53.1, C54.1, C59.1, C63.1, C64.1, D8.1 (K), Q10.2 (S), Q13.2 (S), Q5.2 (S), R29.1, U3.7 (GND); no longer C2.2, Q3.2 (S), U2.6 (VSS)
- removed net +BAT: R30.1, U6.2 (OUT)
Other:
- moved on the sheet: C64, Q3, Q5

Commit message: Bom
Parts:
- removed D13, D8: 1N4148W, Diode_SMD:D_SOD-123, symbol Diode:1N4148W
- removed Q3, Q5: CMSN3416K-HF, Package_TO_SOT_SMD:SOT-23, symbol Transistor_FET:BSS123
- added D13, D8: 1N4148WS, Diode_SMD:D_SOD-323, symbol Diode:1N4148WS
- added Q3, Q5: AO3400A, Package_TO_SOT_SMD:SOT-23, symbol Transistor_FET:AO3400A
- C2: footprint Resistor_SMD:R_0603_1608Metric_Pad0.98x0.95mm_HandSolder -> Capacitor_SMD:C_0603_1608Metric_Pad1.08x0.95mm_HandSolder; LCSC (none) -> C14663
- Q2: LCSC (none) -> C2145
- R25, R36: LCSC (none) -> C25804
- R26: value 330 -> 1k; LCSC (none) -> C21190
- R29: LCSC (none) -> C13167
- R30: LCSC (none) -> C23138
Connections:
- net -BATT: now also C2.1, D13.1 (K), Q3.2 (S); no longer C2.2
- net Earth: now also R25.2, R36.2, D8.1 (K), Q5.2 (S); no longer R25.1, R36.1
- net at R30.2, U2.5 (VDD): now also C2.2; no longer C2.1
- net at C27.2, Q10.1 (G): now also D8.2 (A)
- net at C42.2, Q14.1 (G): now also D13.2 (A)
- net at U2.1 (DO): now also Q3.1 (G)
- net at U2.3 (CO): now also Q5.1 (G)
- net at U6.1 (TS): now also R25.1; no longer R25.2
- net at U6.4 (ISET): now also R36.1; no longer R36.2
- new net: Q3.3 (D), Q5.3 (D)
